Commit message: update robot model

File: Chapter09/panda_description/urdf/panda.urdf.xacro (robot description, xacro)
@@ -89,5 +89,5 @@
   </xacro:if>
   <gazebo>
-    <plugin filename="ign_ros2_control-system" name="ign_ros2_control::IgnitionROS2ControlPlugin">
+    <plugin filename="gz_ros2_control-system" name="gz_ros2_control::GazeboSimROS2ControlPlugin">
       <parameters>$(find panda_moveit_config)/config/ros2_controllers.yaml</parameters>
     </plugin>

File: Chapter09/panda_description/urdf/panda_arm.xacro (robot description, xacro)
@@ -6,5 +6,7 @@
   <!--                   -->
   <xacro:include filename="$(find panda_description)/urdf/panda_utils.xacro"/>
+  <!--
   <xacro:include filename="$(find panda_moveit_config)/config/panda.ros2_control.xacro"/>
+  -->
   <xacro:arg name="use_nominal_extrinsics" default="true"/>
   <xacro:arg name="add_plug" default="false" />
@@ -345,5 +347,7 @@
     gazebo_preserve_fixed_joint="${gazebo_preserve_fixed_joint}"
     />
+    <!--
     <xacro:panda_ros2_control name="FakeSystem" initial_positions_file="$(find panda_moveit_config)/config/initial_positions.yaml"/>
+    -->
     <xacro:sensor_d435 parent="${prefix}${link0_name}" use_nominal_extrinsics="$(arg use_nominal_extrinsics)" add_plug="$(arg add_plug)" use_mesh="$(arg use_mesh)">
         <origin xyz="0.1 0.0 0.05" rpy="0 0.0 0" />
@@ -415,9 +419,23 @@
                 <command_interface name="position"/>
                 <state_interface name="position">
+                  <param name="initial_value">-0.78</param>
+                </state_interface>
+                <state_interface name="velocity"/>
+            </joint>
+            <joint name="joint3">
+                <command_interface name="position"/>
+                <state_interface name="position">
                   <param name="initial_value">0.0</param>
                 </state_interface>
                 <state_interface name="velocity"/>
             </joint>
-            <joint name="joint3">
+            <joint name="joint4">
+                <command_interface name="position"/>
+                <state_interface name="position">
+                  <param name="initial_value">-2.35</param>
+                </state_interface>
+                <state_interface name="velocity"/>
+            </joint>
+            <joint name="joint5">
                 <command_interface name="position"/>
                 <state_interface name="position">
@@ -426,22 +444,8 @@
                 <state_interface name="velocity"/>
             </joint>
-            <joint name="joint4">
-                <command_interface name="position"/>
-                <state_interface name="position">
-                  <param name="initial_value">0.0</param>
-                </state_interface>
-                <state_interface name="velocity"/>
-            </joint>
-            <joint name="joint5">
-                <command_interface name="position"/>
-                <state_interface name="position">
-                  <param name="initial_value">0.0</param>
-                </state_interface>
-                <state_interface name="velocity"/>
-            </joint>
             <joint name="joint6">
                 <command_interface name="position"/>
                 <state_interface name="position">
-                  <param name="initial_value">0.0</param>
+                  <param name="initial_value">1.57</param>
                 </state_interface>
                 <state_interface name="velocity"/>
@@ -450,5 +454,5 @@
                 <command_interface name="position"/>
                 <state_interface name="position">
-                  <param name="initial_value">0.0</param>
+                  <param name="initial_value">0.78</param>
                 </state_interface>
                 <state_interface name="velocity"/>

File: Chapter09/panda_moveit_config/config/panda.ros2_control.xacro (robot description, xacro)
@@ -2,9 +2,9 @@
 <robot xmlns:xacro="http://www.ros.org/wiki/xacro">
     <xacro:macro name="panda_ros2_control" params="name initial_positions_file">
-        <xacro:property name="initial_positions" value="${xacro.load_yaml(initial_positions_file)['initial_positions']}"/>
-        <ros2_control name="IgnitionSystem" type="system">
+        <xacro:property name="initial_positions" value="${load_yaml(initial_positions_file)['initial_positions']}"/>
+        <ros2_control name="${name}" type="system">
             <hardware>
                 <!-- By default, set up controllers for simulation. This won't work on real hardware -->
-                     <plugin>ign_ros2_control/IgnitionSystem</plugin>
+                <plugin>mock_components/GenericSystem</plugin>
             </hardware>
             <joint name="joint1">
@@ -57,18 +57,4 @@
                 <state_interface name="velocity"/>
             </joint>
-            <joint name="finger_joint1">
-                <command_interface name="position"/>
-                <state_interface name="position">
-                  <param name="initial_value">${initial_positions['finger_joint1']}</param>
-                </state_interface>
-                <state_interface name="velocity"/>
-            </joint>
-            <joint name="finger_joint2">
-                <command_interface name="position"/>
-                <state_interface name="position">
-                  <param name="initial_value">${initial_positions['finger_joint2']}</param>
-                </state_interface>
-                <state_interface name="velocity"/>
-            </joint>
         </ros2_control>
     </xacro:macro>

Commit message: update chapter 09

File: Chapter09/panda_description/urdf/panda.urdf.xacro (robot description, xacro)
@@ -90,5 +90,5 @@
   <gazebo>
     <plugin filename="gz_ros2_control-system" name="gz_ros2_control::GazeboSimROS2ControlPlugin">
-      <parameters>$(find panda_moveit_config)/config/ros2_controllers.yaml</parameters>
+      <parameters>$(find panda_description)/config/ros2_controllers.yaml</parameters>
     </plugin>
   </gazebo>

File: Chapter09/panda_description/urdf/panda_arm.xacro (robot description, xacro)
@@ -400,9 +400,9 @@
           </noise>
         </camera>
-          <plugin filename="libignition-gazebo-sensors-system.so" name="ignition::gazebo::systems::Sensors">
+          <plugin filename="libgz-sim-sensors-system.so" name="gz::sim::systems::Sensors">
             <render_engine>ogre</render_engine>
           </plugin>
       </sensor>
-    </gazebo>
+      </gazebo>
    <ros2_control name="2DofPosition" type="system">
         <hardware>

File: Chapter09/panda_moveit_config/config/panda.ros2_control.xacro (robot description, xacro)
@@ -2,5 +2,5 @@
 <robot xmlns:xacro="http://www.ros.org/wiki/xacro">
     <xacro:macro name="panda_ros2_control" params="name initial_positions_file">
-        <xacro:property name="initial_positions" value="${load_yaml(initial_positions_file)['initial_positions']}"/>
+        <xacro:property name="initial_positions" value="${xacro.load_yaml(initial_positions_file)['initial_positions']}"/>
         <ros2_control name="${name}" type="system">
             <hardware>
